File: kicad/daedalus.kicad_pcb (KiCad board)
At the start: 4 copper layers, 42 x 50.2 mm, 98 parts, among them J1 CAN Bus, J2 CAN Bus, J5 A Terminal, J6 B Terminal, J7 C Terminal, J9 USB_B_Micro, Q1 AO3401A, U1 XT30, U10 TPH, U11 TPH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

Commit message: Added gerber files and centroid file
Parts:
- added G***: LOGO, daedalus_kicad_lib:daedalus, B.Cu at (143.9, 85.8)
